File: padd/padd.kicad_sch (KiCad schematic)
At the start: 71 parts, among them SW1 RotaryEncoder_Switch, SW2 RotaryEncoder_Switch, U1 Elite-C

Commit message: move to rp2040 onboard
Parts:
- removed U1: Elite-C, PCM_marbastlib-xp-promicroish:Elite-C_ACH, symbol PCM_marbastlib-promicroish:Elite-C
- added C1, C2: 10u, Capacitor_SMD:C_0402_1005Metric, symbol Device:C_Small
- added C10, C11, C12, C13, C3, C4, C5, C7, C8, C9: 100n, Capacitor_SMD:C_0402_1005Metric, symbol Device:C_Small
- added C14, C6: 1u, Capacitor_SMD:C_0402_1005Metric, symbol Device:C_Small
- added C15, C16: 22p, Capacitor_SMD:C_0402_1005Metric, symbol Device:C_Small
- added F1: 500mA, Fuse:Fuse_1206_3216Metric, symbol Device:Fuse_Small
- added J1: USB_C_Receptacle_USB2.0, Connector_USB:USB_C_Receptacle_HRO_TYPE-C-31-M-12, symbol Connector:USB_C_Receptacle_USB2.0
- added R1, R5: 1k, Resistor_SMD:R_0402_1005Metric, symbol Device:R_Small
- added R2, R3: 5.1k, Resistor_SMD:R_0402_1005Metric, symbol Device:R_Small
- added R4: DNF, Resistor_SMD:R_0402_1005Metric, symbol Device:R_Small
- added R6: 220, Resistor_SMD:R_0402_1005Metric, symbol Device:R_Small
- added SW1: SW_Push, Button_Switch_SMD:SW_Push_1P1T_NO_6x6mm_H9.5mm, symbol Switch:SW_Push
- added U1: RP2040, Package_DFN_QFN:QFN-56-1EP_7x7mm_P0.4mm_EP3.2x3.2mm, symbol MCU_RaspberryPi:RP2040
- added U2: W25Q128JVS, Package_SO:SOIC-8_5.23x5.23mm_P1.27mm, symbol Memory_Flash:W25Q128JVS
- added U3: SRV05-4, PCM_marbastlib-various:SOT-23-6-routable, symbol PCM_marbastlib-various:SRV05-4
- added U4: XC6206PxxxMR, PCM_marbastlib-various:SOT-23-6-routable, symbol Regulator_Linear:XC6206PxxxMR
- added Y1: Crystal_GND24_Small, Crystal:Crystal_SMD_2016-4Pin_2.0x1.6mm, symbol Device:Crystal_GND24_Small
- D1, D10, D11, D12, D13, D14, D15, D16, D17, D18, D19, D2, D20, D21, D22, D3, D4, D5, D6, D7, D8, D9: footprint Diode_SMD:D_0402_1005Metric_Pad0.77x0.64mm_HandSolder -> Diode_SMD:D_0402_1005Metric
- renumbered SW1 to ENC1, SW2 to ENC2
Connections:
- net COL5 is gone; now on net COL4: MX10.1, MX15.1, MX20.1, MX5.1
- net +5V: now also C1.1, F1.2, U3.5 (VP), U4.3 (VI)
- net COL2: now also MX13.1, MX18.1, MX3.1, MX8.1; no longer MX12.1, MX17.1, MX2.1, MX21.1, MX7.1
- net COL3: now also MX14.1, MX19.1, MX22.1, MX4.1, MX9.1; no longer MX13.1, MX18.1, MX3.1, MX8.1
- net COL4: no longer MX14.1, MX19.1, MX22.1, MX4.1, MX9.1
- net GND: now also C1.2, C10.2, C11.2, C12.2, C13.2, C14.2, C15.1, C16.1, C2.2, C3.2, C4.2, C5.2, C6.2, C7.2, C8.2, C9.2, J1.A1 (GND), J1.A12 (GND), J1.B1 (GND), J1.B12 (GND), J1.S1 (SHIELD), R2.2, R3.1, SW1.2, U1.19 (TESTEN), U1.57 (GND), U2.4 (GND), U3.2 (VN), U4.1 (GND), Y1.2, Y1.4
- net LED_R3_DOUT: now reaches LED20.2 (DOUT), LED21.3 (DIN)
- net LED_R1_DOUT: now reaches LED10.2 (DOUT), LED11.3 (DIN)
- net LED_R0_DOUT: now reaches LED5.2 (DOUT), LED6.3 (DIN)
- net LED_R2_DOUT: now reaches LED15.2 (DOUT), LED16.3 (DIN)
- net LED_DIN: no longer names the net of LED1.3 (DIN)
- net LED_DIN: now also R6.2
- new net: J1.A5 (CC1), R2.1
- new net: J1.B5 (CC2), R3.2
- new net +1V1: C4.1, C5.1, C6.1, U1.23 (DVDD), U1.45 (VREG_VOUT), U1.50 (DVDD)
- new net +3V3: C10.1, C11.1, C12.1, C13.1, C14.1, C2.1, C3.1, C7.1, C8.1, C9.1, R1.2, R4.2, U1.1 (IOVDD), U1.10 (IOVDD), U1.22 (IOVDD), U1.33 (IOVDD), U1.42 (IOVDD), U1.43 (ADC_AVDD), U1.44 (VREG_IN), U1.48 (USB_VDD), U1.49 (IOVDD), U2.8 (VCC), U4.2 (VO)
- new net COL1: MX12.1, MX17.1, MX2.1, MX21.1, MX7.1
- new net D+: J1.A7 (D-), J1.B7 (D-), U1.47 (USB_DP), U3.3 (IO2)
- new net D-: J1.A6 (D+), J1.B6 (D+), U1.46 (USB_DM), U3.4 (IO3)
- new net LED_R0_DIN: R6.1
- new net QSPI_SCLK: U1.52 (QSPI_SCLK), U2.6 (CLK)
- new net QSPI_SS: R4.1, R5.2, U1.56 (QSPI_SS), U2.1 (~{CS})
- new net SD0: U1.53 (QSPI_SD0), U2.5 (DI(IO0))
- new net SD1: U1.55 (QSPI_SD1), U2.2 (DO(IO1))
- new net SD2: U1.54 (QSPI_SD2), U2.3 (IO2)
- new net SD3: U1.51 (QSPI_SD3), U2.7 (IO3)
- new net SWCLK: U1.24 (SWCLK)
- new net SWD: U1.25 (SWD)
- new net VBUS: F1.1, J1.A4 (VBUS), J1.A9 (VBUS), J1.B4 (VBUS), J1.B9 (VBUS)
- new net XIN: C15.2, U1.20 (XIN), Y1.3
- new net XOUT: C16.2, U1.21 (XOUT), Y1.1
- new net ~{RESET}: R1.1, U1.26 (RUN)
- new net ~{USB_BOOT}: R5.1, SW1.1
- no-connect marks 0 -> 2
Other:
- moved on the sheet: D1, D10, D11, D12, D13, D14, D15, D16, D17, D18, D19, D2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
